Commit message: Fix different joint limit unit between a1 and aliengo

File: unitree_description/urdf/a1/const.xacro (robot description, xacro)
@@ -30,14 +30,14 @@
     <xacro:property name="damping" value="0"/>
     <xacro:property name="friction" value="0"/>
-    <xacro:property name="hip_max" value="46"/>
-    <xacro:property name="hip_min" value="-46"/>
+    <xacro:property name="hip_max" value="${46*pi/180.0}"/>
+    <xacro:property name="hip_min" value="${-46*pi/180.0}"/>
     <xacro:property name="hip_velocity_max" value="21"/>
     <xacro:property name="hip_torque_max" value="33.5"/>
-    <xacro:property name="thigh_max" value="240"/>
-    <xacro:property name="thigh_min" value="-60"/>
+    <xacro:property name="thigh_max" value="${240*pi/180.0}"/>
+    <xacro:property name="thigh_min" value="${-60*pi/180.0}"/>
     <xacro:property name="thigh_velocity_max" value="21"/>
     <xacro:property name="thigh_torque_max" value="33.5"/>
-    <xacro:property name="calf_max" value="-52.5"/>
-    <xacro:property name="calf_min" value="-154.5"/>
+    <xacro:property name="calf_max" value="${-52.5*pi/180.0}"/>
+    <xacro:property name="calf_min" value="${-154.5*pi/180.0}"/>
     <xacro:property name="calf_velocity_max" value="21"/>
     <xacro:property name="calf_torque_max" value="33.5"/>

File: unitree_description/urdf/common/gazebo.xacro (robot description, xacro)
@@ -8,21 +8,21 @@
         </plugin>
     </gazebo>
-    <!-- Show the trajectory of trunk center. -->
-    <gazebo>
-        <plugin name="3dplot" filename="libLinkPlot3DPlugin.so">
-            <frequency>10</frequency>
-            <plot>
-                <link>base</link>
-                <pose>0 0 0 0 0 0</pose>
-                <material>Gazebo/Yellow</material>
-            </plot>
-        </plugin>
-    </gazebo>
-    <gazebo>
-        <plugin filename="libgazebo_ros_force.so" name="gazebo_ros_force">
-            <bodyName>trunk</bodyName>
-            <topicName>/apply_force/trunk</topicName>
-        </plugin>
-    </gazebo>
+    <!--    &lt;!&ndash; Show the trajectory of trunk center. &ndash;&gt;-->
+    <!--    <gazebo>-->
+    <!--        <plugin name="3dplot" filename="libLinkPlot3DPlugin.so">-->
+    <!--            <frequency>10</frequency>-->
+    <!--            <plot>-->
+    <!--                <link>base</link>-->
+    <!--                <pose>0 0 0 0 0 0</pose>-->
+    <!--                <material>Gazebo/Yellow</material>-->
+    <!--            </plot>-->
+    <!--        </plugin>-->
+    <!--    </gazebo>-->
+    <!--    <gazebo>-->
+    <!--        <plugin filename="libgazebo_ros_force.so" name="gazebo_ros_force">-->
+    <!--            <bodyName>trunk</bodyName>-->
+    <!--            <topicName>/apply_force/trunk</topicName>-->
+    <!--        </plugin>-->
+    <!--    </gazebo>-->
     <!-- Foot contacts. -->
     <gazebo reference="FR_calf">

File: unitree_description/urdf/common/leg.xacro (robot description, xacro)
@@ -10,10 +10,10 @@
             <dynamics damping="${damping}" friction="${friction}"/>
             <xacro:if value="${(mirror_dae == True)}">
-                <limit effort="${hip_torque_max}" velocity="${hip_velocity_max}" lower="${hip_min*pi/180.0}"
-                       upper="${hip_max*pi/180.0}"/>
+                <limit effort="${hip_torque_max}" velocity="${hip_velocity_max}" lower="${hip_min}"
+                       upper="${hip_max}"/>
             </xacro:if>
             <xacro:if value="${(mirror_dae == False)}">
-                <limit effort="${hip_torque_max}" velocity="${hip_velocity_max}" lower="${-hip_max*pi/180.0}"
-                       upper="${-hip_min*pi/180.0}"/>
+                <limit effort="${hip_torque_max}" velocity="${hip_velocity_max}" lower="${-hip_max}"
+                       upper="${-hip_min}"/>
             </xacro:if>
         </joint>
@@ -72,6 +72,6 @@
             <axis xyz="0 1 0"/>
             <dynamics damping="${damping}" friction="${friction}"/>
-            <limit effort="${thigh_torque_max}" velocity="${thigh_velocity_max}" lower="${thigh_min*pi/180.0}"
-                   upper="${thigh_max*pi/180.0}"/>
+            <limit effort="${thigh_torque_max}" velocity="${thigh_velocity_max}" lower="${thigh_min}"
+                   upper="${thigh_max}"/>
         </joint>
         <link name="${name}_thigh">
@@ -111,6 +111,5 @@
             <axis xyz="0 1 0"/>
             <dynamics damping="${damping}" friction="${friction}"/>
-            <limit effort="${calf_torque_max}" velocity="${calf_velocity_max}" lower="${calf_min*pi/180.0}"
-                   upper="${calf_max*pi/180.0}"/>
+            <limit effort="${calf_torque_max}" velocity="${calf_velocity_max}" lower="${calf_min}" upper="${calf_max}"/>
         </joint>
         <link name="${name}_calf">
