Commit message: Remove trunk link

File: unitree_description/urdf/common/leg.xacro (robot description, xacro)
@@ -5,5 +5,5 @@
         <joint name="${name}_hip_joint" type="revolute">
             <xacro:insert_block name="origin"/>
-            <parent link="trunk"/>
+            <parent link="base_link"/>
             <child link="${name}_hip"/>
             <axis xyz="1 0 0"/>

File: unitree_description/urdf/robot.xacro (robot description, xacro)
@@ -11,21 +11,8 @@
             <origin rpy="0 0 0" xyz="0 0 0"/>
             <parent link="world"/>
-            <child link="base"/>
+            <child link="base_link"/>
         </joint>
     </xacro:if>
-    <link name="base">
-        <visual>
-            <origin rpy="0 0 0" xyz="0 0 0"/>
-            <geometry>
-                <box size="0.001 0.001 0.001"/>
-            </geometry>
-        </visual>
-    </link>
-    <joint name="floating_base" type="fixed">
-        <origin rpy="0 0 0" xyz="0 0 0"/>
-        <parent link="base"/>
-        <child link="trunk"/>
-    </joint>
-    <link name="trunk">
+    <link name="base_link">
         <visual>
             <origin rpy="0 0 0" xyz="0 0 0"/>

Commit message: Rename "name of leg" to "prefix"

File: unitree_description/urdf/common/leg.xacro (robot description, xacro)
@@ -2,9 +2,9 @@
 <robot xmlns:xacro="http://www.ros.org/wiki/xacro">
     <xacro:include filename="$(find unitree_description)/urdf/common/transmission.xacro"/>
-    <xacro:macro name="leg" params="name mirror mirror_dae front_hind front_hind_dae *origin">
-        <joint name="${name}_hip_joint" type="revolute">
+    <xacro:macro name="leg" params="prefix mirror mirror_dae front_hind front_hind_dae *origin">
+        <joint name="${prefix}_hip_joint" type="revolute">
             <xacro:insert_block name="origin"/>
             <parent link="base_link"/>
-            <child link="${name}_hip"/>
+            <child link="${prefix}_hip"/>
             <axis xyz="1 0 0"/>
             <dynamics damping="${damping}" friction="${friction}"/>
@@ -18,5 +18,5 @@
             </xacro:if>
         </joint>
-        <link name="${name}_hip">
+        <link name="${prefix}_hip">
             <visual>
                 <xacro:if value="${(mirror_dae == True) and (front_hind_dae == True)}">
@@ -52,11 +52,11 @@
             </inertial>
         </link>
-        <joint name="${name}_hip_fixed" type="fixed">
+        <joint name="${prefix}_hip_fixed" type="fixed">
             <origin rpy="0 0 0" xyz="0 ${(thigh_shoulder_length/2.0+hip_offset)*mirror} 0"/>
-            <parent link="${name}_hip"/>
-            <child link="${name}_thigh_shoulder"/>
+            <parent link="${prefix}_hip"/>
+            <child link="${prefix}_thigh_shoulder"/>
         </joint>
         <!-- this link is only for collision -->
-        <link name="${name}_thigh_shoulder">
+        <link name="${prefix}_thigh_shoulder">
             <collision>
                 <origin rpy="${pi/2.0} 0 0" xyz="0 0 0"/>
@@ -66,8 +66,8 @@
             </collision>
         </link>
-        <joint name="${name}_thigh_joint" type="revolute">
+        <joint name="${prefix}_thigh_joint" type="revolute">
             <origin rpy="0 0 0" xyz="0 ${thigh_offset*mirror} 0"/>
-            <parent link="${name}_hip"/>
-            <child link="${name}_thigh"/>
+            <parent link="${prefix}_hip"/>
+            <child link="${prefix}_thigh"/>
             <axis xyz="0 1 0"/>
             <dynamics damping="${damping}" friction="${friction}"/>
@@ -75,5 +75,5 @@
                    upper="${thigh_max}"/>
         </joint>
-        <link name="${name}_thigh">
+        <link name="${prefix}_thigh">
             <visual>
                 <origin rpy="0 0 0" xyz="0 0 0"/>
@@ -105,13 +105,13 @@
             </inertial>
         </link>
-        <joint name="${name}_calf_joint" type="revolute">
+        <joint name="${prefix}_calf_joint" type="revolute">
             <origin rpy="0 0 0" xyz="0 0 ${-thigh_length}"/>
-            <parent link="${name}_thigh"/>
-            <child link="${name}_calf"/>
+            <parent link="${prefix}_thigh"/>
+            <child link="${prefix}_calf"/>
             <axis xyz="0 1 0"/>
             <dynamics damping="${damping}" friction="${friction}"/>
             <limit effort="${calf_torque_max}" velocity="${calf_velocity_max}" lower="${calf_min}" upper="${calf_max}"/>
         </joint>
-        <link name="${name}_calf">
+        <link name="${prefix}_calf">
             <visual>
                 <origin rpy="0 0 0" xyz="0 0 0"/>
@@ -136,10 +136,10 @@
             </inertial>
         </link>
-        <joint name="${name}_foot_fixed" type="fixed">
+        <joint name="${prefix}_foot_fixed" type="fixed">
             <origin rpy="0 0 0" xyz="0 0 ${-(calf_length)}"/>
-            <parent link="${name}_calf"/>
-            <child link="${name}_foot"/>
+            <parent link="${prefix}_calf"/>
+            <child link="${prefix}_foot"/>
         </joint>
-        <link name="${name}_foot">
+        <link name="${prefix}_foot">
             <visual>
                 <origin rpy="0 0 0" xyz="0 0 0"/>
@@ -163,5 +163,5 @@
             </inertial>
         </link>
-        <xacro:leg_transmission name="${name}"/>
+        <xacro:leg_transmission name="${prefix}"/>
     </xacro:macro>
 </robot>

File: unitree_description/urdf/common/transmission.xacro (robot description, xacro)
@@ -2,32 +2,32 @@
 <robot xmlns:xacro="http://www.ros.org/wiki/xacro">
     <xacro:macro name="leg_transmission" params="name">
-        <transmission name="${name}_hip_tran">
+        <transmission name="${prefix}_hip_tran">
             <type>transmission_interface/SimpleTransmission</type>
-            <joint name="${name}_hip_joint">
-            <hardwareInterface>hardware_interface/EffortJointInterface</hardwareInterface>
+            <joint name="${prefix}_hip_joint">
+                <hardwareInterface>hardware_interface/EffortJointInterface</hardwareInterface>
             </joint>
-            <actuator name="${name}_hip_motor">
-            <hardwareInterface>hardware_interface/EffortJointInterface</hardwareInterface>
-            <mechanicalReduction>1</mechanicalReduction>
+            <actuator name="${prefix}_hip_motor">
+                <hardwareInterface>hardware_interface/EffortJointInterface</hardwareInterface>
+                <mechanicalReduction>1</mechanicalReduction>
             </actuator>
         </transmission>
-        <transmission name="${name}_thigh_tran">
+        <transmission name="${prefix}_thigh_tran">
             <type>transmission_interface/SimpleTransmission</type>
-            <joint name="${name}_thigh_joint">
-            <hardwareInterface>hardware_interface/EffortJointInterface</hardwareInterface>
+            <joint name="${prefix}_thigh_joint">
+                <hardwareInterface>hardware_interface/EffortJointInterface</hardwareInterface>
             </joint>
-            <actuator name="${name}_thigh_motor">
-            <hardwareInterface>hardware_interface/EffortJointInterface</hardwareInterface>
-            <mechanicalReduction>1</mechanicalReduction>
+            <actuator name="${prefix}_thigh_motor">
+                <hardwareInterface>hardware_interface/EffortJointInterface</hardwareInterface>
+                <mechanicalReduction>1</mechanicalReduction>
             </actuator>
         </transmission>
-        <transmission name="${name}_calf_tran">
+        <transmission name="${prefix}_calf_tran">
             <type>transmission_interface/SimpleTransmission</type>
-            <joint name="${name}_calf_joint">
-            <hardwareInterface>hardware_interface/EffortJointInterface</hardwareInterface>
+            <joint name="${prefix}_calf_joint">
+                <hardwareInterface>hardware_interface/EffortJointInterface</hardwareInterface>
             </joint>
-            <actuator name="${name}_calf_motor">
-            <hardwareInterface>hardware_interface/EffortJointInterface</hardwareInterface>
-            <mechanicalReduction>1</mechanicalReduction>
+            <actuator name="${prefix}_calf_motor">
+                <hardwareInterface>hardware_interface/EffortJointInterface</hardwareInterface>
+                <mechanicalReduction>1</mechanicalReduction>
             </actuator>
         </transmission>

File: unitree_description/urdf/robot.xacro (robot description, xacro)
@@ -36,14 +36,14 @@
         </inertial>
     </link>
-    <xacro:leg name="FR" mirror="-1" mirror_dae="False" front_hind="1" front_hind_dae="True">
+    <xacro:leg prefix="FR" mirror="-1" mirror_dae="False" front_hind="1" front_hind_dae="True">
         <origin rpy="0 0 0" xyz="${leg_offset_x} ${-leg_offset_y} 0"/>
     </xacro:leg>
-    <xacro:leg name="FL" mirror="1" mirror_dae="True" front_hind="1" front_hind_dae="True">
+    <xacro:leg prefix="FL" mirror="1" mirror_dae="True" front_hind="1" front_hind_dae="True">
         <origin rpy="0 0 0" xyz="${leg_offset_x} ${leg_offset_y} 0"/>
     </xacro:leg>
-    <xacro:leg name="RR" mirror="-1" mirror_dae="False" front_hind="-1" front_hind_dae="False">
+    <xacro:leg prefix="RR" mirror="-1" mirror_dae="False" front_hind="-1" front_hind_dae="False">
         <origin rpy="0 0 0" xyz="${-leg_offset_x} ${-leg_offset_y} 0"/>
     </xacro:leg>
-    <xacro:leg name="RL" mirror="1" mirror_dae="True" front_hind="-1" front_hind_dae="False">
+    <xacro:leg prefix="RL" mirror="1" mirror_dae="True" front_hind="-1" front_hind_dae="False">
         <origin rpy="0 0 0" xyz="${-leg_offset_x} ${leg_offset_y} 0"/>
     </xacro:leg>
