Commit message: Add bbq_gazebo

File: unitree_description/urdf/common/gazebo.xacro (robot description, xacro)
@@ -103,13 +103,8 @@
         </visual>
     </gazebo>
-    <gazebo reference="base">
-        <material>Gazebo/Green</material>
-        <turnGravityOff>false</turnGravityOff>
-    </gazebo>
-    <gazebo reference="trunk">
-        <mu1>0.2</mu1>
-        <mu2>0.2</mu2>
-        <kp value="1000000.0"/>
-        <kd value="1.0"/>
+    <gazebo reference="base_link">
+        <maxVel>100.</maxVel>
+        <kp>10000.</kp>
+        <kd>0.</kd>
     </gazebo>
     <gazebo reference="stick_link">

Commit message: Add unitree_imu to gazebo hardware_interface

File: unitree_description/urdf/common/gazebo.xacro (robot description, xacro)
@@ -20,21 +20,4 @@
         </plugin>
     </gazebo>
-    <!--    &lt;!&ndash; Show the trajectory of trunk center. &ndash;&gt;-->
-    <!--    <gazebo>-->
-    <!--        <plugin name="3dplot" filename="libLinkPlot3DPlugin.so">-->
-    <!--            <frequency>10</frequency>-->
-    <!--            <plot>-->
-    <!--                <link>base</link>-->
-    <!--                <pose>0 0 0 0 0 0</pose>-->
-    <!--                <material>Gazebo/Yellow</material>-->
-    <!--            </plot>-->
-    <!--        </plugin>-->
-    <!--    </gazebo>-->
-    <!--    <gazebo>-->
-    <!--        <plugin filename="libgazebo_ros_force.so" name="gazebo_ros_force">-->
-    <!--            <bodyName>trunk</bodyName>-->
-    <!--            <topicName>/apply_force/trunk</topicName>-->
-    <!--        </plugin>-->
-    <!--    </gazebo>-->
     <!-- Foot contacts. -->
     <gazebo reference="FR_calf">
@@ -113,5 +96,5 @@
         <material>Gazebo/White</material>
     </gazebo>
-    <gazebo reference="imu_link">
+    <gazebo reference="unitree_imu">
         <mu1>0.2</mu1>
         <mu2>0.2</mu2>

File: unitree_description/urdf/robot.xacro (robot description, xacro)
@@ -5,4 +5,5 @@
     <xacro:include filename="$(find unitree_description)/urdf/common/leg.xacro"/>
     <xacro:include filename="$(find unitree_description)/urdf/common/gazebo.xacro"/>
+    <xacro:include filename="$(find unitree_description)/urdf/common/imu.xacro"/>
     <xacro:include filename="$(find unitree_description)/urdf/$(arg robot_type)/const.xacro"/>
     <xacro:if value="$(arg hung_up)">
@@ -36,29 +37,5 @@
         </inertial>
     </link>
-    <joint name="unitree_imu_joint" type="fixed">
-        <parent link="base_link"/>
-        <child link="unitree_imu"/>
-        <origin rpy="0 0 0" xyz="0 0 0"/>
-    </joint>
-    <link name="unitree_imu">
-        <inertial>
-            <mass value="0.001"/>
-            <origin rpy="0 0 0" xyz="0 0 0"/>
-            <inertia ixx="0.0001" ixy="0" ixz="0" iyy="0.000001" iyz="0" izz="0.0001"/>
-        </inertial>
-        <visual>
-            <origin rpy="0 0 0" xyz="0 0 0"/>
-            <geometry>
-                <box size="0.001 0.001 0.001"/>
-            </geometry>
-            <material name="red"/>
-        </visual>
-        <collision>
-            <origin rpy="0 0 0" xyz="0 0 0"/>
-            <geometry>
-                <box size=".001 .001 .001"/>
-            </geometry>
-        </collision>
-    </link>
+    <xacro:IMU connected_to="base_link" imu_name="unitree_imu" xyz="0. 0. 0." rpy="0. 0. 0."/>
     <xacro:leg prefix="FR" mirror="-1" mirror_dae="False" front_hind="1" front_hind_dae="True">
         <origin rpy="0 0 0" xyz="${leg_offset_x} ${-leg_offset_y} 0"/>

Commit message: Add odom pub to StateEstimateBase

File: unitree_description/urdf/common/gazebo.xacro (robot description, xacro)
@@ -96,9 +96,4 @@
         <material>Gazebo/White</material>
     </gazebo>
-    <gazebo reference="unitree_imu">
-        <mu1>0.2</mu1>
-        <mu2>0.2</mu2>
-        <material>Gazebo/Red</material>
-    </gazebo>
     <!-- FL leg -->
     <gazebo reference="FL_hip">
