Commit message: Add aliengo

File: unitree_description/urdf/robot.xacro (robot description, xacro)
@@ -33,5 +33,4 @@
                 <mesh filename="package://unitree_description/meshes/$(arg robot_type)/trunk.dae" scale="1 1 1"/>
             </geometry>
-            <material name="orange"/>
         </visual>
         <collision>

Commit message: Add unitree_imu link

File: unitree_description/urdf/robot.xacro (robot description, xacro)
@@ -36,4 +36,29 @@
         </inertial>
     </link>
+    <joint name="unitree_imu_joint" type="fixed">
+        <parent link="base_link"/>
+        <child link="unitree_imu"/>
+        <origin rpy="0 0 0" xyz="0 0 0"/>
+    </joint>
+    <link name="unitree_imu">
+        <inertial>
+            <mass value="0.001"/>
+            <origin rpy="0 0 0" xyz="0 0 0"/>
+            <inertia ixx="0.0001" ixy="0" ixz="0" iyy="0.000001" iyz="0" izz="0.0001"/>
+        </inertial>
+        <visual>
+            <origin rpy="0 0 0" xyz="0 0 0"/>
+            <geometry>
+                <box size="0.001 0.001 0.001"/>
+            </geometry>
+            <material name="red"/>
+        </visual>
+        <collision>
+            <origin rpy="0 0 0" xyz="0 0 0"/>
+            <geometry>
+                <box size=".001 .001 .001"/>
+            </geometry>
+        </collision>
+    </link>
     <xacro:leg prefix="FR" mirror="-1" mirror_dae="False" front_hind="1" front_hind_dae="True">
         <origin rpy="0 0 0" xyz="${leg_offset_x} ${-leg_offset_y} 0"/>
