Commit message: Remove link and joint only for leg hip collision

File: unitree_description/urdf/aliengo/const.xacro (robot description, xacro)
@@ -10,5 +10,5 @@
     <xacro:property name="hip_length" value="0.0418"/>
     <xacro:property name="thigh_shoulder_radius" value="0.044"/>
-    <xacro:property name="thigh_shoulder_length" value="0.08"/>
+    <xacro:property name="thigh_shoulder_length" value="0.03"/>
     <xacro:property name="thigh_width" value="0.0374"/>
     <xacro:property name="thigh_height" value="0.043"/>

File: unitree_description/urdf/common/leg.xacro (robot description, xacro)
@@ -52,18 +52,4 @@
             </inertial>
         </link>
-        <joint name="${prefix}_hip_fixed" type="fixed">
-            <origin rpy="0 0 0" xyz="0 ${(thigh_shoulder_length/2.0+hip_offset)*mirror} 0"/>
-            <parent link="${prefix}_hip"/>
-            <child link="${prefix}_thigh_shoulder"/>
-        </joint>
-        <!-- this link is only for collision -->
-        <link name="${prefix}_thigh_shoulder">
-            <collision>
-                <origin rpy="${pi/2.0} 0 0" xyz="0 0 0"/>
-                <geometry>
-                    <cylinder length="${thigh_shoulder_length}" radius="${thigh_shoulder_radius}"/>
-                </geometry>
-            </collision>
-        </link>
         <joint name="${prefix}_thigh_joint" type="revolute">
             <origin rpy="0 0 0" xyz="0 ${thigh_offset*mirror} 0"/>
@@ -94,4 +80,10 @@
                 <geometry>
                     <box size="${thigh_length} ${thigh_width} ${thigh_height}"/>
+                </geometry>
+            </collision>
+            <collision>
+                <origin rpy="${pi/2.0} 0 0" xyz="0 0 0"/>
+                <geometry>
+                    <cylinder length="${thigh_shoulder_length}" radius="${thigh_shoulder_radius}"/>
                 </geometry>
             </collision>

Commit message: Add inaccurate damping and friction to aliengo

File: unitree_description/urdf/aliengo/const.xacro (robot description, xacro)
@@ -28,6 +28,6 @@
     <xacro:property name="hip_offset" value="0.083"/>
     <!-- joint limits -->
-    <xacro:property name="damping" value="0"/>
-    <xacro:property name="friction" value="0"/>
+    <xacro:property name="damping" value="0.05"/>
+    <xacro:property name="friction" value="0.01"/>
     <xacro:property name="hip_max" value="${70*pi/180.0}"/>
     <xacro:property name="hip_min" value="${-70*pi/180.0}"/>

Commit message: Correct dynamics parameters

File: unitree_description/urdf/aliengo/const.xacro (robot description, xacro)
@@ -19,9 +19,9 @@
     <xacro:property name="stick_length" value="0.2"/>
     <!-- kinematic value -->
-    <xacro:property name="thigh_offset" value="0.083"/>
+    <xacro:property name="thigh_offset" value="0.0868"/>
     <xacro:property name="thigh_length" value="0.25"/>
     <xacro:property name="calf_length" value="0.25"/>
     <!-- leg offset from trunk center value -->
-    <xacro:property name="leg_offset_x" value="0.2399"/>
+    <xacro:property name="leg_offset_x" value="0.2407"/>
     <xacro:property name="leg_offset_y" value="0.051"/>
     <xacro:property name="trunk_offset_z" value="0.01675"/>
@@ -33,14 +33,14 @@
     <xacro:property name="hip_min" value="${-70*pi/180.0}"/>
     <xacro:property name="hip_velocity_max" value="20"/>
-    <xacro:property name="hip_torque_max" value="44"/>
+    <xacro:property name="hip_torque_max" value="35.278"/>
     <xacro:property name="thigh_max" value="1e10"/>
     <xacro:property name="thigh_min" value="-1e10"/>
     <xacro:property name="thigh_velocity_max" value="20"/>
-    <xacro:property name="thigh_torque_max" value="44"/>
+    <xacro:property name="thigh_torque_max" value="35.278"/>
     <xacro:property name="calf_max" value="${-37*pi/180.0}"/>
     <xacro:property name="calf_min" value="${-159*pi/180.0}"/>
-    <xacro:property name="calf_velocity_max" value="16"/>
-    <xacro:property name="calf_torque_max" value="55"/>
-    <!-- dynamics inertial value -->
+    <xacro:property name="calf_velocity_max" value="15.89"/>
+    <xacro:property name="calf_torque_max" value="44.4"/>
+    <!-- dynamics inertial value    total 22.0kg-->
     <!-- trunk -->
     <xacro:property name="trunk_mass" value="11.041"/>
